File: dicebug.kicad_pcb (KiCad board)
At the start: 2 copper layers, 47.3 x 40.9 mm, 32 parts, among them SW1 SW_SPDT, U1 74LV163ADR, U3 74HCS7266DR, U5 iqs211a

Commit message: WIP
Parts:
- added C1: 47n, Capacitor_SMD:C_0805_2012Metric, F.Cu at (96.0, 103.0)
- added R8: 47k, Resistor_SMD:R_0805_2012Metric, F.Cu at (105.9, 102.5)
- R13: value 100k -> 47k
- moved R5 6.74 mm to (85.2, 108.1), turned to -90 degrees
- moved R13 4.62 mm to (92.7, 107.0), turned to -90 degrees
- moved C7 1.69 mm to (89.7, 110.0)
Connections:
- R13 pad 2: Net-(U5-IO2/SDA) -> Net-(U1-CP)
- TP4 pad 1: Net-(U5-IO2/SDA) -> Net-(U1-CP)
- U1 pad 1: +3V0 -> Net-(U1-~{MR})
- U3 pad 1: Net-(U5-IO2/SDA) -> Net-(C1-Pad1)
- U3 pad 3: Net-(U1-CP) -> Net-(U1-~{MR})
- U5 pad 3: Net-(U5-IO2/SDA) -> Net-(U1-CP)
Routing:
- net Net-(U5-IO2/SDA): track 15.0 -> 0.00 mm
- net GND: track 131.2 -> 144.6 mm
- net Net-(U1-~{MR}): track 0.00 -> 9.40 mm
- net Net-(C1-Pad1): track 0.00 -> 9.26 mm
- net Net-(R4-Pad1): track 87.7 -> 80.8 mm
- net Net-(D5-A): track 5.93 -> 11.6 mm
- net Net-(R2-Pad1): track 78.2 -> 83.4 mm
- net Net-(U1-CP): track 10.2 -> 15.0 mm
- net +3V0: track 54.4 -> 58.0 mm
- net Net-(R6-Pad1): track 41.1 -> 42.9 mm
- net Net-(U1-Q0): track 36.6 -> 38.4 mm
- net Net-(U5-VREG): track 6.12 -> 4.96 mm
- net Net-(JP5-C): track 0.99 -> 0.00 mm

Commit message: WIP: integrating artwork
Parts:
- removed JP5: sel_half, Connector_PinHeader_1.27mm:PinHeader_1x03_P1.27mm_Vertical
- moved TP6 66.1 mm to (103.0, 113.6)
- moved TP4 15.7 mm to (134.9, 118.3)
Connections:
- TP6 pad 1: Net-(JP5-C) -> GND
Routing:
- net GND: track 144.6 -> 146.3 mm, vias 0 -> 1
- added copper zone on B.Cu, net GND
- removed copper zone on B.Cu, net Net-(JP5-C)
Other:
- board size 47.3 x 40.9 mm -> 120.6 x 77.6 mm
